Commit message: fix issues

File: omni_description/urdf/omni.urdf (robot description, URDF)
Before this commit: robot phantom_omni, 7 links, 6 joints
Joints:
- joint elbow: origin xyz=0.0075 .134 0 rpy=-1.5 0 0 -> xyz=0.0075 0.134 0 rpy=-1.5 0 0
- joint roll: axis 0 1 0 -> 0 -1 0
- joint shoulder: origin xyz=-0.0075 0 0.035 rpy=0 0 0 -> xyz=-0.0075 0 0.035
- joint waist: origin xyz=0 0 0.09 rpy=0 0 0 -> xyz=0 0 0.09
